File: hypergolic V1.3/hypergolic_right.kicad_pcb (KiCad board)
At the start: 2 copper layers, 118.3 x 87.7 mm, 25 parts, among them SW10 SW_Push, SW11 SW_Push, SW12 SW_Push, SW14 SW_Push, SW15 SW_Push, SW16 SW_Push, SW17 SW_Push, SW18 SW_Push, SW2 SW_Push, SW20 SW_Push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

Commit message: flip left power switch and add plate file
Parts:
- SW_POWER1: moved to F.Cu
- turned SW_POWER1 to 0 degrees
Routing:
- net BT+: track 77.1 -> 81.3 mm, vias 0 -> 1
- net raw: track 49.0 -> 46.5 mm, vias 0 -> 1
- net gnd: vias 12 -> 8
